File: USB-PD-PoE.sch (KiCad schematic (older format))
At the start: 134 parts, among them J1 8P8C_Shielded, J2 8P8C_Shielded, J3 TagConnect_TC2030_SWD, J4 USB_C_Receptacle_USB2.0, Q1 FDC2512, Q2 2N7002, Q3 2N7002, Q4 2N7002, Q5 APM4953KC, Q6 2N7002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

Commit message: Fix ethernet transformer footprint
Parts:
- U1: LCSC C8735 -> C46034
Changed lines of the file:
@@
 F 2 "Package_QFP:LQFP-64_10x10mm_P0.5mm" H -4300 3050 50  0001 R CNN
 F 3 "http://www.st.com/st-web-ui/static/active/en/resource/technical/document/datasheet/CD00161566.pdf" H -3700 4750 50  0001 C CNN
-F 4 "C8735" H -3700 4750 50  0001 C CNN "LCSC"
+F 4 "C46034" H -3700 4750 50  0001 C CNN "LCSC"
 	1    -3700 4750
 	1    0    0    -1

Commit message: Optimize design for manufacturing
Replace components not available at JLC anymore.
Parts:
- removed U8: SY8303, Package_TO_SOT_SMD:SOT-23-8, symbol Regulator_Switching_Silergy:SY8303
- added C41: 4.7uF, Capacitor_SMD:C_0402_1005Metric, symbol Device:C_Small
- added U10: SY8368, Package_QFN_Silergy:QFN_3x3-10_SY8368, symbol Regulator_Switching_Silergy:SY8368
- C2, C34: LCSC C134761 -> C249868
- J1, J2: footprint Connector_RJ_Ckmtw:Connector_8P8C_R-RJ45R08P-B000 -> Connector_RJ_Ckmtw:Connector_8P8C_R-RJ45R08P-C000; LCSC C386756 -> C386757
- R28: value 100kR -> 10kR; LCSC C25741 -> C25744
- R3: value 1.6kR -> 300R; LCSC C25931 -> C25102
- R31: value 110kR -> 100kR; footprint Resistor_SMD:R_0603_1608Metric -> Resistor_SMD:R_0402_1005Metric; LCSC C25805 -> C25741
- R6: value 4.3kR -> 5.6kR; LCSC C23159 -> C25908
- R9: value 402R -> 390R; footprint Resistor_SMD:R_0402_1005Metric -> Resistor_SMD:R_0603_1608Metric; LCSC C41042 -> C23151
Connections:
- net +12V: now also U10.7 (IN), U10.8 (IN)
- net BUCK_EN: now also U10.1 (EN)
- net BUCK_OUT: now also R28.2; no longer R31.1
- net GND: now also C41.2, U10.3 (ILMT), U10.9 (GND); no longer R28.2
- net at C29.2, R32.1, R35.1: now also R31.1, U10.4 (FB); no longer R31.2
- net at R28.1: now also R31.2
- net at C28.1, L3.1: now also U10.10 (LX)
- net at C28.2: now also U10.6 (BS)
- new net: C41.1, U10.5 (VC)
Other:
- moved on the sheet: C28, R27
Changed lines of the file:
@@
 F 0 "J2" H 1507 6517 50  0000 C CNN
 F 1 "8P8C_Shielded" H 1507 6426 50  0000 C CNN
-F 2 "Connector_RJ_Ckmtw:Connector_8P8C_R-RJ45R08P-B000" V 1450 5875 50  0001 C CNN
+F 2 "Connector_RJ_Ckmtw:Connector_8P8C_R-RJ45R08P-C000" V 1450 5875 50  0001 C CNN
 F 3 "~" V 1450 5875 50  0001 C CNN
-F 4 "C386756" H 1450 5850 50  0001 C CNN "LCSC"
+F 4 "C386757" H 1450 5850 50  0001 C CNN "LCSC"
 	1    1450 5850
 	1    0    0    -1
@@
 F 0 "J1" H 5707 6517 50  0000 C CNN
 F 1 "8P8C_Shielded" H 5707 6426 50  0000 C CNN
-F 2 "Connector_RJ_Ckmtw:Connector_8P8C_R-RJ45R08P-B000" V 5650 5875 50  0001 C CNN
+F 2 "Connector_RJ_Ckmtw:Connector_8P8C_R-RJ45R08P-C000" V 5650 5875 50  0001 C CNN
 F 3 "~" V 5650 5875 50  0001 C CNN
-F 4 "C386756" H 5650 5850 50  0001 C CNN "LCSC"
+F 4 "C386757" H 5650 5850 50  0001 C CNN "LCSC"
 	1    5650 5850
 	-1   0    0    -1
@@
 P 1800 1950
 F 0 "R3" H 1730 1904 50  0000 R CNN
-F 1 "1.6kR" H 1730 1995 50  0000 R CNN
+F 1 "300R" H 1730 1995 50  0000 R CNN
 F 2 "Resistor_SMD:R_0402_1005Metric" V 1730 1950 50  0001 C CNN
 F 3 "~" H 1800 1950 50  0001 C CNN
-F 4 "C25931" H 1800 1950 50  0001 C CNN "LCSC"
+F 4 "C25102" H 1800 1950 50  0001 C CNN "LCSC"
 	1    1800 1950
 	-1   0    0    1
@@
 P 2200 2300
 F 0 "R6" V 2407 2300 50  0000 C CNN
-F 1 "4.3kR" V 2316 2300 50  0000 C CNN
+F 1 "5.6kR" V 2316 2300 50  0000 C CNN
 F 2 "Resistor_SMD:R_0603_1608Metric" V 2130 2300 50  0001 C CNN
 F 3 "~" H 2200 2300 50  0001 C CNN
-F 4 "C23159" H 2200 2300 50  0001 C CNN "LCSC"
+F 4 "C25908" H 2200 2300 50  0001 C CNN "LCSC"
 	1    2200 2300
 	0    -1   -1   0
@@
 F 2 "Capacitor_SMD:CP_Elec_6.3x7.7" H 3338 650 50  0001 C CNN
 F 3 "~" H 3300 800 50  0001 C CNN
-F 4 "C134761" H 3300 800 50  0001 C CNN "LCSC"
+F 4 "C249868" H 3300 800 50  0001 C CNN "LCSC"
 	1    3300 800
 	1    0    0    -1
@@
 P 3800 1900
 F 0 "R9" V 3593 1900 50  0000 C CNN
-F 1 "402R" V 3684 1900 50  0000 C CNN
-F 2 "Resistor_SMD:R_0402_1005Metric" V 3730 1900 50  0001 C CNN
+F 1 "390R" V 3684 1900 50  0000 C CNN
+F 2 "Resistor_SMD:R_0603_1608Metric" V 3730 1900 50  0001 C CNN
 F 3 "~" H 3800 1900 50  0001 C CNN
-F 4 "C41042" V 3800 1900 50  0001 C CNN "LCSC"
+F 4 "C23151" V 3800 1900 50  0001 C CNN "LCSC"
 	1    3800 1900
 	0    1    1    0
@@
 NoConn ~ -3900 2950
 $Comp
-L Regulator_Switching_Silergy:SY8303 U8
-U 1 1 616EB067
-P 14550 4850
-F 0 "U8" H 14350 5300 50  0000 C CNN
-F 1 "SY8303" H 14550 4850 50  0000 C CNN
-F 2 "Package_TO_SOT_SMD:SOT-23-8" H 14550 4850 50  0001 C CNN
-F 3 "https://datasheet.lcsc.com/szlcsc/Silergy-Corp-SY8303AIC_C97054.pdf" H 14550 4850 50  0001 C CNN
-F 4 "C97054" H 14550 5439 50  0001 C CNN "LCSC"
-	1    14550 4850
-	1    0    0    -1
-$EndComp
-$Comp
 L Device:L L3
 U 1 1 616EC9F3
@@
 L Device:C C28
 U 1 1 6172916C
-P 14750 4300
-F 0 "C28" V 14498 4300 50  0000 C CNN
-F 1 "10nF" V 14589 4300 50  0000 C CNN
-F 2 "Capacitor_SMD:C_0402_1005Metric" H 14788 4150 50  0001 C CNN
-F 3 "~" H 14750 4300 50  0001 C CNN
-F 4 "C15195" V 14750 4300 50  0001 C CNN "LCSC"
-	1    14750 4300
+P 14750 4250
+F 0 "C28" V 14498 4250 50  0000 C CNN
+F 1 "10nF" V 14589 4250 50  0000 C CNN
+F 2 "Capacitor_SMD:C_0402_1005Metric" H 14788 4100 50  0001 C CNN
+F 3 "~" H 14750 4250 50  0001 C CNN
+F 4 "C15195" V 14750 4250 50  0001 C CNN "LCSC"
+	1    14750 4250
 	0    1    1    0
 $EndComp
 Wire Wire Line
-	14950 4600 15000 4600
-Wire Wire Line
-	15000 4600 15000 4300
+	15000 4250 14900 4250
 Wire Wire Line
-	15000 4300 14900 4300
-Connection ~ 15000 4600
-Wire Wire Line
-	15000 4600 15050 4600
+	14600 4250 14550 4250
 Wire Wire Line
-	14600 4300 14550 4300
-Wire Wire Line
-	14550 4300 14550 4350
-$Comp
-L Device:R_Small R31
-U 1 1 617A409A
-P 15400 4750
-F 0 "R31" H 15459 4796 50  0000 L CNN
-F 1 "110kR" H 15459 4705 50  0000 L CNN
-F 2 "Resistor_SMD:R_0603_1608Metric" H 15400 4750 50  0001 C CNN
-F 3 "~" H 15400 4750 50  0001 C CNN
-F 4 "C25805" H 15400 4750 50  0001 C CNN "LCSC"
-	1    15400 4750
-	1    0    0    -1
-$EndComp
+	14550 4250 14550 4300
 $Comp
 L Device:C_Small C29
@@
 	15600 5800 15700 5800
 Wire Wire Line
-	15400 4850 15400 4900
-Wire Wire Line
 	15400 4900 15700 4900
 Wire Wire Line
@@
 	15700 5850 15700 5800
 Wire Wire Line
-	15400 4650 15400 4600
-Wire Wire Line
 	15400 4600 15350 4600
 Wire Wire Line
@@
 Wire Wire Line
 	15100 4900 15400 4900
-Text Label 13800 5100 0    50   ~ 0
+Text Label 13800 4850 0    50   ~ 0
 BUCK_EN
 Wire Wire Line
-	13800 5100 14100 5100
-Wire Wire Line
-	14100 5100 14100 5150
-Connection ~ 14100 5100
-Wire Wire Line
-	14100 5100 14150 5100
+	13800 4850 13950 4850
 $Comp
 L power:GND #PWR06
@@
 $EndComp
 Wire Wire Line
-	14550 5400 14100 5400
-Wire Wire Line
-	14100 5400 14100 5350
-Wire Wire Line
-	14550 5400 14550 5350
-Connection ~ 14550 5400
-Wire Wire Line
-	14550 5450 14550 5400
+	13950 5400 13950 5350
 $Comp
 L Device:C_Small C23
@@
 Connection ~ 13700 4600
 $Comp
-L Device:R_Small R28
-U 1 1 61C4CAC6
-P 15000 5250
-F 0 "R28" H 15059 5296 50  0000 L CNN
-F 1 "100kR" H 15059 5205 50  0000 L CNN
-F 2 "Resistor_SMD:R_0402_1005Metric" H 15000 5250 50  0001 C CNN
-F 3 "~" H 15000 5250 50  0001 C CNN
-F 4 "C25741" H 15000 5250 50  0001 C CNN "LCSC"
-	1    15000 5250
-	1    0    0    -1
-$EndComp
-Wire Wire Line
-	14950 5100 15000 5100
-Wire Wire Line
-	15000 5100 15000 5150
-Wire Wire Line
-	14550 5400 15000 5400
-Wire Wire Line
-	15000 5400 15000 5350
-$Comp
 L Device:R_Small R27
 U 1 1 61CDA267
-P 14100 5250
-F 0 "R27" H 14159 5296 50  0000 L CNN
-F 1 "100kR" H 14159 5205 50  0000 L CNN
-F 2 "Resistor_SMD:R_0402_1005Metric" H 14100 5250 50  0001 C CNN
-F 3 "~" H 14100 5250 50  0001 C CNN
-F 4 "C25741" H 14100 5250 50  0001 C CNN "LCSC"
-	1    14100 5250
+P 13950 5250
+F 0 "R27" H 14009 5296 50  0000 L CNN
+F 1 "100kR" H 14009 5205 50  0000 L CNN
+F 2 "Resistor_SMD:R_0402_1005Metric" H 13950 5250 50  0001 C CNN
+F 3 "~" H 13950 5250 50  0001 C CNN
+F 4 "C25741" H 13950 5250 50  0001 C CNN "LCSC"
+	1    13950 5250
 	-1   0    0    1
 $EndComp
@@
 F 2 "Capacitor_SMD:CP_Elec_6.3x7.7" H 17338 2500 50  0001 C CNN
 F 3 "~" H 17300 2650 50  0001 C CNN
-F 4 "C134761" H 17300 2650 50  0001 C CNN "LCSC"
+F 4 "C249868" H 17300 2650 50  0001 C CNN "LCSC"
 	1    17300 2650
 	1    0    0    -1
@@
 Wire Wire Line
 	-2700 5150 -3000 5150
+$Comp
+L Regulator_Switching_Silergy:SY8368 U10
+U 1 1 6087FB35
+P 14550 5000
+F 0 "U10" H 14550 5881 50  0000 C CNN
+F 1 "SY8368" H 14550 5790 50  0000 C CNN
+F 2 "Package_QFN_Silergy:QFN_3x3-10_SY8368" H 14750 4950 50  0001 C CNN
+F 3 "https://datasheet.lcsc.com/szlcsc/Silergy-Corp-SY8368QNC_C125897.pdf" H 14550 5000 50  0001 C CNN
+F 4 "C125897" H 14550 5000 50  0001 C CNN "LCSC"
+	1    14550 5000
+	1    0    0    -1
+$EndComp
+Wire Wire Line
+	14950 4600 15000 4600
+Wire Wire Line
+	13950 5150 13950 4850
+Connection ~ 13950 4850
+Wire Wire Line
+	14550 5350 14550 5400
+Wire Wire Line
+	13950 4850 14150 4850
+Wire Wire Line
+	13950 5400 14050 5400
+Connection ~ 14550 5400
+Wire Wire Line
+	14550 5400 14550 5450
+Wire Wire Line
+	14150 5100 14050 5100
+Wire Wire Line
+	14050 5100 14050 5400
+Connection ~ 14050 5400
+Wire Wire Line
+	14050 5400 14550 5400
+$Comp
+L Device:C_Small C41
+U 1 1 60B8A1BE
+P 15000 5250
+F 0 "C41" H 15092 5296 50  0000 L CNN
+F 1 "4.7uF" H 15092 5205 50  0000 L CNN
+F 2 "Capacitor_SMD:C_0402_1005Metric" H 15000 5250 50  0001 C CNN
+F 3 "~" H 15000 5250 50  0001 C CNN
+F 4 "C23733" H 15000 5250 50  0001 C CNN "LCSC"
+	1    15000 5250
+	1    0    0    -1
+$EndComp
+Wire Wire Line
+	14550 5400 15000 5400
+Wire Wire Line
+	15000 5400 15000 5350
+Wire Wire Line
+	14950 5100 15000 5100
+Wire Wire Line
+	15000 5100 15000 5150
+Wire Wire Line
+	15000 4250 15000 4600
+Connection ~ 15000 4600
+Wire Wire Line
+	15000 4600 15050 4600
+$Comp
+L Device:R_Small R28
+U 1 1 60D91269
+P 15300 4700
+F 0 "R28" H 15370 4746 50  0000 L CNN
+F 1 "10kR" H 15370 4655 50  0000 L CNN
+F 2 "Resistor_SMD:R_0402_1005Metric" V 15230 4700 50  0001 C CNN
+F 3 "~" H 15300 4700 50  0001 C CNN
+F 4 "C25744" H 15300 4700 50  0001 C CNN "LCSC"
+	1    15300 4700
+	0    -1   -1   0
+$EndComp
+$Comp
+L Device:R_Small R31
+U 1 1 60DDFD85
+P 15300 4800
+F 0 "R31" H 15359 4846 50  0000 L CNN
+F 1 "100kR" H 15359 4755 50  0000 L CNN
+F 2 "Resistor_SMD:R_0402_1005Metric" H 15300 4800 50  0001 C CNN
+F 3 "~" H 15300 4800 50  0001 C CNN
+F 4 "C25741" H 15300 4800 50  0001 C CNN "LCSC"
+	1    15300 4800
+	0    1    1    0
+$EndComp
+Wire Wire Line
+	15200 4800 15200 4700
+Wire Wire Line
+	15400 4600 15400 4700
+Wire Wire Line
+	15400 4800 15400 4900
 $EndSCHEMATC
